File: Asservissement_CDFR_2023/Asservissement_CDFR_2023.kicad_pcb (KiCad board)
At the start: 2 copper layers, 86 x 114 mm, 117 parts, among them IC1 A3930KJPTR-T, IC2 A3930KJPTR-T, J1 Connecteur batterie, J10 Free Connecteur, J11 Conn_01x02, J12 Conn_01x02, J13 Connecteur Odométrie, J2 Conn_01x03, J3 Conn_01x05, J4 Connecteur Programmation, J5 Conn_01x03, J6 Connecteur Odométrie, J7 Conn_01x03, J8 Conn_01x03, J9 Conn_01x05, Q1 QM6006D, Q10 QM6006D, Q11 QM6006D, Q12 QM6006D, Q13 Q_NMOS_GDS, Q2 QM6006D, Q3 QM6006D, Q4 QM6006D, Q5 QM6006D, Q6 QM6006D, Q7 QM6006D, Q8 QM6006D, Q9 QM6006D, U1 LM317_SOT-223, U2 TPS562200, U3 STM32F401RCTx, Y1 Crystal_GND24

Commit message: Routing almost done
Parts:
- added H1: MountingHole_Pad, MountingHole:MountingHole_3.2mm_M3_Pad_Via, F.Cu at (117.3, 34.0)
- added H2: MountingHole_Pad, MountingHole:MountingHole_3.2mm_M3_Pad_Via, F.Cu at (61.6, 140.6)
- added H3: MountingHole_Pad, MountingHole:MountingHole_3.2mm_M3_Pad_Via, F.Cu at (61.6, 34.0)
- added H4: MountingHole_Pad, MountingHole:MountingHole_3.2mm_M3_Pad_Via, F.Cu at (117.3, 140.8)
- added H5: MountingHole_Pad, MountingHole:MountingHole_2.7mm_Pad_Via, F.Cu at (94.6, 34.0)
- added H6: MountingHole_Pad, MountingHole:MountingHole_2.7mm_Pad_Via, F.Cu at (38.5, 113.0)
- added H7: MountingHole_Pad, MountingHole:MountingHole_2.7mm_Pad_Via, F.Cu at (38.6, 60.5)
- added H8: MountingHole_Pad, MountingHole:MountingHole_2.7mm_Pad_Via, F.Cu at (94.6, 140.6)
- added kibuzzard-637D40DA: G***, kibuzzard-637D40DA, F.Cu at (44.4, 119.8)
- added kibuzzard-637D40E8: G***, kibuzzard-637D40E8, F.Cu at (50.3, 126.0)
- added kibuzzard-637D40F4: G***, kibuzzard-637D40F4, F.Cu at (46.8, 121.2)
- added kibuzzard-637D40F4: G***, kibuzzard-637D40F4, F.Cu at (52.8, 127.2)
- added kibuzzard-637D4198: G***, kibuzzard-637D4198, F.Cu at (80.6, 133.2)
- added kibuzzard-637D41A9: G***, kibuzzard-637D41A9, F.Cu at (81.5, 72.2)
- added kibuzzard-637D41F7: G***, kibuzzard-637D41F7, F.Cu at (50.5, 102.7)
- added kibuzzard-637D4204: G***, kibuzzard-637D4204, F.Cu at (52.1, 104.7)
- added kibuzzard-637D4217: G***, kibuzzard-637D4217, F.Cu at (48.7, 101.0)
- added kibuzzard-637D428D: G***, kibuzzard-637D428D, F.Cu at (37.0, 96.5)
- added kibuzzard-637D42B7: G***, kibuzzard-637D42B7, F.Cu at (44.7, 73.8)
- added kibuzzard-637D42C2: G***, kibuzzard-637D42C2, F.Cu at (44.7, 76.2)
- added kibuzzard-637D42CB: G***, kibuzzard-637D42CB, F.Cu at (44.8, 78.5)
- added kibuzzard-637D42F0: G***, kibuzzard-637D42F0, F.Cu at (51.6, 66.7)
- added kibuzzard-637D4301: G***, kibuzzard-637D4301, F.Cu at (51.0, 69.0)
- added kibuzzard-637D4322: G***, kibuzzard-637D4322, F.Cu at (50.7, 71.5)
- added kibuzzard-637D4331: G***, kibuzzard-637D4331, F.Cu at (50.9, 74.2)
- added kibuzzard-637D436E: G***, kibuzzard-637D436E, F.Cu at (68.5, 34.0)
- added kibuzzard-637D4374: G***, kibuzzard-637D4374, F.Cu at (78.5, 33.6)
- added kibuzzard-637D437D: G***, kibuzzard-637D437D, F.Cu at (71.1, 34.0)
- added kibuzzard-637D4386: G***, kibuzzard-637D4386, F.Cu at (73.5, 34.0)
- added kibuzzard-637D438C: G***, kibuzzard-637D438C, F.Cu at (76.1, 34.0)
- added kibuzzard-637D43BC: G***, kibuzzard-637D43BC, F.Cu at (82.4, 38.4)
- added kibuzzard-637D43CD: G***, kibuzzard-637D43CD, F.Cu at (83.1, 98.8)
- added kibuzzard-637D4446: G***, kibuzzard-637D4446, F.Cu at (52.1, 54.2)
- added kibuzzard-637D4446: G***, kibuzzard-637D4446, F.Cu at (47.5, 68.5)
- added kibuzzard-637D4455: G***, kibuzzard-637D4455, F.Cu at (50.2, 56.1)
- added kibuzzard-637D4463: G***, kibuzzard-637D4463, F.Cu at (44.4, 71.2)
- added kibuzzard-637D4463: G***, kibuzzard-637D4463, F.Cu at (49.1, 56.9)
- added kibuzzard-637D44C4: G***, kibuzzard-637D44C4, F.Cu at (39.7, 68.7)
- added kibuzzard-637D44E0: G***, kibuzzard-637D44E0, F.Cu at (51.4, 48.4)
- added kibuzzard-637D4536: G***, kibuzzard-637D4536, F.Cu at (45.6, 70.4)
- added kibuzzard-637D45A0: G***, kibuzzard-637D45A0, F.Cu at (46.5, 69.4)
- added kibuzzard-eD: G***, kibuzzard-637D447D, F.Cu at (51.1, 55.1)
- moved R19 95.3 mm to (59.4, 126.3), turned to -135 degrees
- moved J12 88.2 mm to (56.3, 123.8), turned to 135 degrees
- moved J11 77.9 mm to (50.0, 117.4), turned to 135 degrees
- moved R10 71.0 mm to (46.0, 112.1), turned to 45 degrees
- moved J6 63.2 mm to (49.0, 51.3), turned to -135 degrees
- moved J13 60.9 mm to (48.5, 61.6), turned to -135 degrees
- moved JP1 57.0 mm to (37.2, 84.8), turned to 0 degrees
- moved R32 54.6 mm to (88.3, 39.1), turned to 90 degrees
- moved C26 53.0 mm to (61.5, 93.0)
- moved C25 52.2 mm to (64.0, 96.3), turned to -45 degrees
- moved J7 46.8 mm to (39.2, 73.7), turned to -90 degrees
- moved C20 45.7 mm to (78.3, 76.0), turned to 180 degrees
- moved R38 44.8 mm to (65.0, 128.0), turned to -90 degrees
- moved C15 43.9 mm to (41.0, 97.0), turned to 180 degrees
- moved C14 42.5 mm to (40.2, 94.0), turned to 90 degrees
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Connections:
- C25 pad 1: +5V -> +3.3V
- C26 pad 1: +5V -> +3.3V
- U3 pad 13: +5V -> +3.3V
Routing:
- net +BATT: track 241.6 -> 390.9 mm, vias 3 -> 12
- net GND: track 486.6 -> 618.4 mm, vias 5 -> 8
- net +3.3V: track 58.8 -> 179.4 mm, vias 4 -> 1
- net +5V: track 142.1 -> 204.8 mm
- net Free1: track 62.8 -> 15.5 mm, vias 0 -> 1
- net info_direction_2: track 0.00 -> 46.3 mm
- net disable_2: track 89.1 -> 43.6 mm, vias 2 -> 0
- net Net-(J11-Pad2): track 101.1 -> 56.3 mm, vias 6 -> 1
- net reset_2: track 80.3 -> 38.0 mm, vias 2 -> 0
- net Info_vitesse_2: track 76.7 -> 36.5 mm, vias 4 -> 0
- net Net-(J6-Pad2): track 74.5 -> 35.6 mm, vias 2 -> 0
- net MODE_1: track 80.1 -> 44.9 mm, vias 2 -> 0
- net direction_controle_1: track 0.00 -> 33.0 mm
- net reset_1: track 0.00 -> 29.9 mm
- net Free4: track 58.0 -> 28.2 mm, vias 2 -> 0
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Other:
- board size 86 x 114 mm -> 86.4 x 114.3 mm
