File: Asservissement_CDFR_2023/Asservissement_CDFR_2023.kicad_sch (KiCad schematic)
At the start: 130 parts, among them IC1 A3930KJPTR-T, IC2 A3930KJPTR-T, J1 Connecteur batterie, J10 Free Connecteur, J11 Conn_01x02, J12 Conn_01x02, J13 Connecteur Odométrie, J2 Conn_01x03, J3 Conn_01x05, J4 Connecteur Programmation, J5 Conn_01x03, J6 Connecteur Odométrie, J7 Conn_01x03, J8 Conn_01x03, J9 Conn_01x05, Q1 QM6006D, Q10 QM6006D, Q11 QM6006D, Q12 QM6006D, Q13 Q_NMOS_GDS, Q2 QM6006D, Q3 QM6006D, Q4 QM6006D, Q5 QM6006D, Q6 QM6006D, Q7 QM6006D, Q8 QM6006D, Q9 QM6006D, U1 LM317_SOT-223, U3 STM32F401RCTx, U4 LMR16020PDDA, Y1 Crystal_GND24

Commit message: V4 add button, test point, remove quartz, pot and fix current
Parts:
- removed C14, C15: 10pF, Capacitor_SMD:C_0805_2012Metric_Pad1.18x1.45mm_HandSolder, symbol Device:C
- removed J11, J12: Conn_01x02, Connector_JST:JST_XH_B2B-XH-A_1x02_P2.50mm_Vertical, symbol Connector_Generic:Conn_01x02
- removed R1, R8: 10k, Resistor_SMD:R_0805_2012Metric_Pad1.20x1.40mm_HandSolder, symbol Device:R
- removed RV1, RV2: 10k, Potentiometer_THT:Potentiometer_Bourns_3386C_Horizontal, symbol Device:R_Potentiometer
- removed Y1: Crystal_GND24, Crystal:Crystal_SMD_2520-4Pin_2.5x2.0mm, symbol Device:Crystal_GND24
- added C31: 0.1nF, Capacitor_SMD:C_0805_2012Metric_Pad1.18x1.45mm_HandSolder, symbol Device:C
- added R45: 100k, Resistor_SMD:R_0805_2012Metric_Pad1.20x1.40mm_HandSolder, symbol Device:R
- added SW1, SW2, SW3: SW_Push, Button_Switch_THT:SW_PUSH_6mm_H5mm, symbol Switch:SW_Push
- added TP1, TP10, TP11, TP12, TP13, TP14, TP2, TP25, TP26, TP27, TP28, TP29, TP3, TP30, TP31, TP32, TP33, TP34, TP35, TP36, TP4, TP5, TP6, TP7, TP8, TP9: TestPoint, TestPoint:TestPoint_Pad_D1.0mm, symbol Connector:TestPoint
- R19: value 10k -> 100k
Connections:
- net +3.3V: now also R10.1, SW1.1, SW2.1, TP14.1
- net +5V: now also R19.2, R45.2, TP13.1
- net Free8: now also U3.44 (PA11); no longer U3.11 (PC3)
- net GND: now also C31.2, SW3.2; no longer R10.1, R19.1
- net Info_erreur_1_1: now also TP29.1
- net Info_erreur_1_2: now also TP11.1
- net Info_erreur_2_1: now also TP30.1
- net Info_erreur_2_2: now also TP12.1
- net Info_vitesse_1: now also TP31.1
- net Info_vitesse_2: now also TP5.1
- net MODE_1: now also TP35.1
- net MODE_2: now also TP2.1
- net action_fault_1: now also TP25.1
- net action_fault_2: now also TP7.1
- net direction_controle_1: now also TP33.1
- net direction_controle_2: now also TP3.1
- net disable_1: now also TP27.1
- net disable_2: now also TP9.1
- net frein_1: now also TP32.1
- net frein_2: now also TP6.1
- net info_direction_1: now also TP26.1
- net info_direction_2: now also TP8.1
- net reset_1: now also TP28.1
- net reset_2: now also TP10.1
- net speed_controle_1: now also TP34.1
- net speed_controle_2: now also TP4.1
- net NRST: now reaches J4.4 (Pin_4), U3.7 (NRST)
- net NRST: now also R10.2, C31.1, SW3.1
- net at U3.52 (PC11): now also SW1.2; no longer R19.2
- net Info_Courant_1_uc: now reaches R34.1, R38.1, U3.15 (PA1)
- net Info_Courant_1_uc: now also TP36.1
- net Info_Courant_2_uc: now reaches R37.1, R39.1
- net Info_Courant_2_uc: now also U3.11 (PC3), TP1.1; no longer U3.44 (PA11)
- net at U3.53 (PC12): now also SW2.2; no longer R10.2
- net at IC1.20 (REF_): now also R19.1
- net at IC2.20 (REF_): now also R45.1
- no-connect marks 13 -> 15
Other:
- moved on the sheet: J10, R34, R37, R38, R39
